Commit message: Restored some motion planning.

File: src/abe_sim/CounterTop/countertop.urdf (robot description, URDF)
Before this commit: robot countertop, 1 links, 0 joints
Links:
- link countertop: geometry collision mesh filename=countertop_collision.obj; visual mesh filename=countertop_collision.obj

File: src/abe_sim/Particle/butterparticle.urdf (robot description, URDF)
Before this commit: robot butterparticle, 1 links, 0 joints
Links:
- link particle: mass 0.01 -> 0.001

File: src/abe_sim/Particle/sugarparticle.urdf (robot description, URDF)
Before this commit: robot sugarparticle, 1 links, 0 joints
Links:
- link particle: mass 0.01 -> 0.001
