Commit message: Incorporated grid-based motion planning.

File: src/abe_sim/Fridge/freezer.urdf (robot description, URDF)
Before this commit: robot fridge, 2 links, 1 joints
Links:
- removed link fridge
- added link freezer, mass 30.0; collision mesh filename=freezer_collision.obj; visual mesh filename=fridge_visual.obj
Joints:
- joint base: child fridge -> freezer

File: src/abe_sim/KitchenCabinet/kitchencabinet.urdf (robot description, URDF)
Before this commit: robot countertop, 1 links, 0 joints
Links:
- link kitchencabinet: geometry collision mesh filename=kitchencabinet_collision.obj; visual mesh filename=kitchencabinet_collision.obj
