Commit message: Pick-place (fetching)

File: src/abe_sim/Abe/abe.urdf (robot description, URDF)
Before this commit: robot abe, 19 links, 18 joints
Joints:
- joint base_y_to_base_yaw: limit effort=1000 velocity=100 -> effort=1000 velocity=6.

Commit message: Pour portioning, now with 2 bowls.

File: src/abe_sim/Abe/abe.urdf (robot description, URDF)
Before this commit: robot abe, 19 links, 18 joints
Joints:
- joint base_x_to_base_y: limit lower=-5 upper=5 effort=1000.0 velocity=3. -> lower=-15 upper=15 effort=1000.0 velocity=3.
- joint hand_left_base_to_hand_left_x: limit lower=-0.5 upper=2 effort=1000.0 velocity=3. -> lower=-0.85 upper=2 effort=1000.0 velocity=3.
- joint hand_left_x_to_hand_left_y: limit lower=-0.5 upper=1.5 effort=1000.0 velocity=3. -> lower=-1.4 upper=1.85 effort=1000.0 velocity=3.
- joint hand_right_base_to_hand_right_x: limit lower=-0.5 upper=2 effort=1000.0 velocity=3. -> lower=-0.85 upper=2 effort=1000.0 velocity=3.
- joint hand_right_x_to_hand_right_y: limit lower=-1.5 upper=0.5 effort=1000.0 velocity=3. -> lower=-1.85 upper=1.4 effort=1000.0 velocity=3.
- joint world_to_base_x: limit lower=-5 upper=5 effort=1000.0 velocity=3. -> lower=-15 upper=15 effort=1000.0 velocity=3.

Commit message: Cookie recipe actions

File: src/abe_sim/Abe/abe.urdf (robot description, URDF)
Before this commit: robot abe, 19 links, 18 joints
Joints:
- joint hand_left_base_to_hand_left_x: limit lower=-0.85 upper=2 effort=1000.0 velocity=3. -> lower=-0.85 upper=2.5 effort=1000.0 velocity=3.
- joint hand_right_base_to_hand_right_x: limit lower=-0.85 upper=2 effort=1000.0 velocity=3. -> lower=-0.85 upper=2.5 effort=1000.0 velocity=3.

File: src/abe_sim/Whisk/whisk.urdf (robot description, URDF)
Before this commit: robot whisk, 2 links, 1 joints
Links:
- link whisk: geometry collision mesh filename=whisk_collision.obj; visual mesh filename=whisk_visual.obj
