Commit message: Demo custom dynamics.

File: 3DObjects/Bread/bread.urdf (robot description, URDF)
Before this commit: robot cooking_knife, 2 links, 1 joints
Links:
- removed link blade
- removed link handle
- added link core, mass 0.2; collision mesh filename=loaf_core.obj; visual mesh filename=loaf_core.obj
- added link crust, mass 0.02; collision mesh filename=loaf_crust.obj; visual mesh filename=loaf_crust.obj
Joints:
- removed joint handle_to_blade
- added joint core_to_crust: type fixed, parent core, child crust, origin xyz=0 0 -0.011 rpy=0 0 0

File: 3DObjects/Bread/bread_slice.urdf (robot description, URDF)
Before this commit: robot cooking_knife, 2 links, 1 joints
Links:
- removed link blade
- removed link handle
- added link core, mass 0.02; collision mesh filename=slice_core.obj; visual mesh filename=slice_core.obj
- added link crust, mass 0.002; collision mesh filename=slice_crust.obj; visual mesh filename=slice_crust.obj
Joints:
- removed joint handle_to_blade
- added joint core_to_crust: type fixed, parent core, child crust, origin xyz=0 0 -0.011 rpy=0 0 0

File: 3DObjects/CookingKnife/buttered_cooking_knife.urdf (robot description, URDF)
Before this commit: robot cooking_knife, 2 links, 1 joints
Links:
- added link butter, mass 0.01; collision mesh filename=butter.obj; visual mesh filename=butter.obj
Joints:
- added joint handle_to_butter: type fixed, parent handle, child butter, origin xyz=0.322 0.013 0 rpy=0 0 0

File: 3DObjects/Egg/cracked_eggshell_flat_half.urdf (robot description, URDF)
Before this commit: robot eggshell_flat_half, 1 links, 0 joints
Links:
- removed link eggshell_flat_half
- added link eggshell, mass 0.0025; collision mesh filename=eggshell_flat_half_collision.obj; visual mesh filename=eggshell_flat_half_visual.obj

File: 3DObjects/Egg/cracked_eggshell_pointy_half.urdf (robot description, URDF)
Before this commit: robot eggshell_pointy_half, 1 links, 0 joints
Links:
- removed link eggshell_pointy_half
- added link egg, mass 0.0025; collision mesh filename=eggshell_pointy_half_collision.obj; visual mesh filename=eggshell_pointy_half_visual.obj

File: 3DObjects/PepperShaker/pepper_particle.urdf (robot description, URDF)
Before this commit: robot peeled_potato, 1 links, 0 joints
Links:
- removed link potato
- added link pepper_particle, mass 0.001; collision mesh filename=pepper_particle.obj; visual mesh filename=pepper_particle.obj
