Commit message: Added various new models, urdf files and modified objectknowledge and processknowledge accordingly

File: src/abe_sim/3DObjects/Banana/bananaPeel.urdf (robot description, URDF)
Before this commit: robot bananaPeel, 1 links, 0 joints
Links:
- link peel: geometry collision mesh filename=peelCollider.obj; visual mesh filename=bananaPeel.obj

File: src/abe_sim/3DObjects/Carrot/carrotPeel.urdf (robot description, URDF)
Before this commit: robot carrotPeel, 1 links, 0 joints
Links:
- link peel: geometry collision mesh filename=carrotPeelCollider.obj; visual mesh filename=carrotPeel.obj
