Commit message: Added some furniture and walls to the kitchen

File: src/abe_sim/3DObjects/Banana/banana.urdf (robot description, URDF)
Before this commit: robot banana, 3 links, 2 joints
Joints:
- joint body_to_nub: origin xyz=0 0.159 0.30377 rpy=0 0 0 -> xyz=0 0.079694 0.1517 rpy=0 0 0
- joint body_to_stem: origin xyz=0 0.159 -0.275 rpy=0 0 0 -> xyz=0 0.078995 -0.137653 rpy=0 0 0

File: src/abe_sim/3DObjects/PottedPlant/pottedPlant.urdf (robot description, URDF)
Before this commit: robot frying_pan, 2 links, 1 joints
Links:
- removed link grip
- removed link pan
- added link plant, mass 0.000; collision mesh filename=pottedPlantPlantCollider.obj; visual mesh filename=pottedPlantPlant.obj
- added link pot, mass 0.00; collision mesh filename=pottedPlantPotCollider.obj; visual mesh filename=pottedPlantPot.obj
Joints:
- removed joint pan_to_grip
- added joint pot_to_plant: type fixed, parent pot, child plant, origin xyz=0 0 1.33481 rpy=0 0 0

File: src/abe_sim/3DObjects/Wall/wall_north.urdf (robot description, URDF)
Before this commit: robot floor, 1 links, 0 joints
Links:
- removed link floor
- added link wall_north, mass 0.00; collision mesh filename=wall_north.obj; visual mesh filename=wall_north.obj

File: src/abe_sim/3DObjects/Wall/wall_south.urdf (robot description, URDF)
Before this commit: robot floor, 1 links, 0 joints
Links:
- removed link floor
- added link wall_south, mass 0.00; collision mesh filename=wall_south.obj; visual mesh filename=wall_south.obj
