Commit message: Salad tests.

File: src/abe_sim/3DObjects/Bacon/bacon.urdf (robot description, URDF)
Before this commit: robot bacon, 3 links, 2 joints
Joints:
- joint body_to_stripe1: origin xyz=-0.02895 0.014182 0 rpy=0 0 0 -> xyz=0.014 0 0.008 rpy=0 0 0
- joint body_to_stripe2: origin xyz=0.03135 0.014182 0 rpy=0 0 0 -> xyz=-0.014 0 0.008 rpy=0 0 0

File: src/abe_sim/3DObjects/Broccoli/broccoli.urdf (robot description, URDF)
Before this commit: robot broccoli, 2 links, 1 joints
Links:
- link head: mass 0.001 -> 0.1; geometry collision mesh filename=broccoliHead.obj; visual mesh filename=broccoliHead.obj
- link stem: mass 0.01 -> 0.05; geometry collision mesh filename=broccoliStem.obj; visual mesh filename=broccoliStem.obj
Joints:
- removed joint stem_to_head
- added joint head_to_stem: type fixed, parent head, child stem, origin xyz=0 0 0 rpy=0 0 0

File: src/abe_sim/3DObjects/CiderVinegar/ciderVinegar.urdf (robot description, URDF)
Before this commit: robot ciderVinegar, 3 links, 2 joints
Links:
- link body: mass 0.02 -> 0.2; geometry collision mesh filename=vinegarBottle.obj; visual mesh filename=vinegarBottle.obj
- link cap: geometry collision mesh filename=vinegarCork.obj; visual mesh filename=vinegarCork.obj
Joints:
- joint body_to_cap: origin xyz=0 0 0.546 rpy=0 0 0 -> xyz=0 0 0.137 rpy=0 0 0
- joint body_to_label: origin xyz=0.069 0 0.225 rpy=0 0 0 -> xyz=0.035 0 -0.029 rpy=0 0 0

File: src/abe_sim/3DObjects/LargeBowl/largebowl.urdf (robot description, URDF)
Before this commit: robot largebowl, 1 links, 0 joints
Links:
- added link handle, mass 0.001; collision mesh filename=handle.obj; visual mesh filename=handle.obj
Joints:
- added joint largebowl_to_handle: type fixed, parent largebowl, child handle, origin xyz=0 -0.26 0.043 rpy=0 0 0

File: src/abe_sim/3DObjects/Mayonnaise/mayonnaise.urdf (robot description, URDF)
Before this commit: robot mayonnaise, 1 links, 0 joints
Links:
- link body: mass 0.01 -> 0.1; geometry collision mesh filename=mayonnaiseBottle.obj; visual mesh filename=mayonnaiseBottle.obj

File: src/abe_sim/3DObjects/Onion/peeledRedOnion.urdf (robot description, URDF)
Before this commit: robot peeled_red_onion, 1 links, 0 joints
Links:
- link peeledRedOnion: mass 0.01 -> 0.09

File: src/abe_sim/3DObjects/Onion/redOnion.urdf (robot description, URDF)
Before this commit: robot redOnion, 1 links, 0 joints
Links:
- link onion: mass 0.01 -> 0.1; geometry collision mesh filename=redOnion.obj; visual mesh filename=redOnion.obj

File: src/abe_sim/3DObjects/Onion/redOnionPeel.urdf (robot description, URDF)
Before this commit: robot red_onion_peel, 1 links, 0 joints
Links:
- link peel: geometry collision mesh filename=redOnionPeelCollider.obj; visual mesh filename=redOnionPeel.obj
