Commit message: Some scale adjustment, cooked bacon, broccoli salad scene.

File: src/abe_sim/3DObjects/Bacon/cookedBacon.urdf (robot description, URDF)
Before this commit: robot bacon, 3 links, 2 joints
Links:
- link body: geometry collision mesh filename=baconCollider.obj; visual mesh filename=CookedBacon.obj
