Commit message: Some mesh updates, a minfix in proc garden for compheight.

File: src/abe_sim/3DObjects/Broccoli/broccoliStem.urdf (robot description, URDF)
Before this commit: robot broccoliStem, 1 links, 0 joints
Links:
- link stem: geometry collision mesh filename=broccoliStem.obj; visual mesh filename=broccoliStem.obj

File: src/abe_sim/3DObjects/KitchenCounter/kitchen_counter.urdf (robot description, URDF)
Before this commit: robot countertop, 2 links, 1 joints
Links:
- link base: geometry collision mesh filename=base_collision.obj; visual mesh filename=base.obj

File: src/abe_sim/3DObjects/LargeBowl/largebowl.urdf (robot description, URDF)
Before this commit: robot largebowl, 2 links, 1 joints
Joints:
- joint largebowl_to_handle: origin xyz=0 -0.26 0.043 rpy=0 0 0 -> xyz=0 -0.207 0.035 rpy=0 0 0

File: src/abe_sim/3DObjects/LargeBowl/largebowlLid.urdf (robot description, URDF)
Before this commit: robot mediumbowlLid, 1 links, 0 joints
Links:
- added link handle, mass 0.01; collision mesh filename=largeLidHandle.obj; visual mesh filename=largeLidHandle.obj
- link lid: geometry collision mesh filename=largeLid.obj; visual mesh filename=largeLid.obj
Joints:
- added joint lid_to_handle: type fixed, parent lid, child handle, origin xyz=0 0 0.044 rpy=0 0 0
