Commit message: Updated hand models for Bea to better match the VR hands

File: src/abe_sim/3DObjects/Bea/bea.urdf (robot description, URDF)
Before this commit: robot bea, 19 links, 18 joints
Links:
- link hand_left_roll: geometry collision mesh filename=bea_left_hand_new.obj; visual mesh filename=bea_left_hand_new.obj
- link hand_right_roll: geometry collision mesh filename=bea_right_hand_new.obj; visual mesh filename=bea_right_hand_new.obj
