Commit message: Updates to proc garden.

File: src/abe_sim/3DObjects/Oven/oven.urdf (robot description, URDF)
Before this commit: robot oven, 11 links, 10 joints
Links:
- link door: geometry collision mesh filename=dummy.obj; visual mesh filename=door.obj
- link handle: geometry collision mesh filename=dummy.obj; visual mesh filename=handle.obj

Commit message: Minfix

File: src/abe_sim/3DObjects/Oven/oven.urdf (robot description, URDF)
Before this commit: robot oven, 11 links, 10 joints
Joints:
- joint base_to_top_back: origin xyz=0 -0.60. 1.35 rpy=0 0 0 -> xyz=0 -0.60 1.35 rpy=0 0 0

Commit message: Temperature setter, adjusting knob for oven.

File: src/abe_sim/3DObjects/Oven/oven.urdf (robot description, URDF)
Before this commit: robot oven, 11 links, 10 joints
Links:
- added link heatknob, mass 0.0; collision mesh filename=heatknob.obj; visual mesh filename=heatknob.obj
- added link heatmarker, mass 0.0; collision mesh filename=heatmarker.obj; visual mesh filename=heatmarker.obj
- added link heatmarkerspots, mass 0.0; collision mesh filename=heatmarkerspots.obj; visual mesh filename=heatmarkerspots.obj
Joints:
- added joint heatmarker_to_heatknob: type revolute, parent heatmarker, child heatknob, origin xyz=0 0 0.03 rpy=0 0 0, axis 0 0 1, limit lower=0 upper=3.141 effort=1000.0 velocity=1.
- added joint heatmarker_to_heatmarkerspots: type fixed, parent heatmarker, child heatmarkerspots, origin xyz=0 0 0.005 rpy=0 0 0
- added joint top_to_heatmarker: type fixed, parent top, child heatmarker, origin xyz=0.91 0.73 0 rpy=-1.57 0 0

Commit message: Fixes for to-preheat-oven

File: src/abe_sim/3DObjects/Oven/oven.urdf (robot description, URDF)
Before this commit: robot oven, 14 links, 13 joints
Links:
- link heatknob: mass 0.0 -> 0.01
