Commit message: Shrink masher and peeled potato models

File: src/abe_sim/3DObjects/Masher/masher.urdf (robot description, URDF)
Before this commit: robot masher, 3 links, 2 joints
Joints:
- joint handle_to_shaft: origin xyz=0.24 0 0 rpy=0 0 0 -> xyz=0.12 0 0 rpy=0 0 0
- joint shaft_to_masher: origin xyz=0.12 0 0 rpy=0 0 0 -> xyz=0.06 0 0 rpy=0 0 0
