Commit message: Broccoli salad tests.

File: src/abe_sim/3DObjects/CiderVinegar/ciderVinegar.urdf (robot description, URDF)
Before this commit: robot ciderVinegar, 3 links, 2 joints
Links:
- added link bottom, mass 0.2; collision mesh filename=bottom.obj; visual mesh filename=bottom.obj
- link body: mass 0.2 -> 0.02
- link label: mass 0.02 -> 0.002
Joints:
- added joint body_to_bottom: type fixed, parent body, child bottom, origin xyz=0 0 -0.06 rpy=0 0 0
- joint body_to_cap: origin xyz=0 0 0.137 rpy=0 0 0 -> xyz=0 0 0.083 rpy=0 0 0
- joint body_to_label: origin xyz=0.035 0 -0.029 rpy=0 0 0 -> xyz=0.034 0 -0.01 rpy=0 0 0

File: src/abe_sim/3DObjects/CuttingBoard/cutting_board.urdf (robot description, URDF)
Before this commit: robot cutting_board, 3 links, 2 joints
Links:
- link edge: geometry collision mesh filename=edgeCollider.obj; visual mesh filename=edge.obj

File: src/abe_sim/3DObjects/Mayonnaise/mayonnaise_jar.urdf (robot description, URDF)
Before this commit: robot mayonnaiseJar, 3 links, 2 joints
Links:
- added link bottom, mass 0.15; collision mesh filename=bottom.obj; visual mesh filename=bottom.obj
Joints:
- added joint jar_to_bottom: type fixed, parent jar, child bottom, origin xyz=0 0 0 rpy=0 0 0
