Commit message: Added new objects
Added chopped green chili pepper, chopped red chili pepper, chocolate chip, chocolate chip bag, chopped cooked chicken, corn, corn can, corn cob,  chopped seeded peeled cucumber slice, cucumber seed, peeled cucumber slice, peeled cucumber, seeded peeled cucumber slice, chopped fresh basil, chopped fresh cilantro, fresh oregano leaf,  minced garlic clove, shredded cabbage, whipped heavy cream particle, chopped seeded half-jalapeno, half jalapeno, jalapeno seed, mango peel

File: src/abe_sim/3DObjects/ChocolateChips/chocolateChip.urdf (robot description, URDF)
Before this commit: robot corn, 1 links, 0 joints
Links:
- removed link corn
- added link chocolateChip, mass 0.001; collision mesh filename=chocolateChip.obj; visual mesh filename=chocolateChip.obj

File: src/abe_sim/3DObjects/ChocolateChips/chocolateChipBag.urdf (robot description, URDF)
Before this commit: robot corn, 1 links, 0 joints
Links:
- removed link corn
- added link chocolate_chip_bag, mass 0.001; collision mesh filename=chocolateChipBag.obj; visual mesh filename=chocolateChipBag.obj

File: src/abe_sim/3DObjects/HeavyCream/whipped_heavy_cream_particle.urdf (robot description, URDF)
Before this commit: robot corn, 1 links, 0 joints
Links:
- removed link corn
- added link whipped_heavy_cream_particle, mass 0.001; collision mesh filename=WhippedHeavyCreamParticle.obj; visual mesh filename=WhippedHeavyCreamParticle.obj
