Commit message: Rescaled objects

File: src/abe_sim/3DObjects/BellPepper/bellPepper.urdf (robot description, URDF)
Before this commit: robot bellPepper, 2 links, 1 joints
Joints:
- joint body_to_stem: origin xyz=0 0.168 0 rpy=0 0 0 -> xyz=0 0.084 0 rpy=0 0 0

File: src/abe_sim/3DObjects/Carrot/carrot.urdf (robot description, URDF)
Before this commit: robot carrot, 2 links, 1 joints
Joints:
- joint fruit_to_tail: origin xyz=0 0.52 0 rpy=0 0 0 -> xyz=0 0.251 0 rpy=0 0 0

File: src/abe_sim/3DObjects/ChiliPepper/chiliGreen.urdf (robot description, URDF)
Before this commit: robot chili, 2 links, 1 joints
Joints:
- joint chi_to_stem: origin xyz=0 0.408695 0 rpy=0 0 0 -> xyz=0 0.2043 0 rpy=0 0 0

File: src/abe_sim/3DObjects/ChiliPepper/chiliRed.urdf (robot description, URDF)
Before this commit: robot chili, 2 links, 1 joints
Joints:
- joint chi_to_stem: origin xyz=0 0.408695 0 rpy=0 0 0 -> xyz=0 0.2043 0 rpy=0 0 0

File: src/abe_sim/3DObjects/Corn/corn.urdf (robot description, URDF)
Before this commit: robot corn, 2 links, 1 joints
Joints:
- joint leaf_to_cob: origin xyz=0 0.196 0 rpy=0 0 0 -> xyz=0 0.098 0 rpy=0 0 0

File: src/abe_sim/3DObjects/ExtraVirginOliveOil/oliveOil.urdf (robot description, URDF)
Before this commit: robot vegetableOil, 3 links, 2 joints
Joints:
- joint body_to_cap: origin xyz=0 0 0.546 rpy=0 0 0 -> xyz=0 0 0.273 rpy=0 0 0
- joint body_to_label: origin xyz=0.069 0 0.225 rpy=0 0 0 -> xyz=0.0345 0 0.1225 rpy=0 0 0

File: src/abe_sim/3DObjects/Jalapeno/jalapeno.urdf (robot description, URDF)
Before this commit: robot jalapeno, 2 links, 1 joints
Joints:
- joint body_to_stem: origin xyz=0 0.26364 0 rpy=0 0 0 -> xyz=0 0.13182 0 rpy=0 0 0

File: src/abe_sim/3DObjects/LimeJuice/limeJuiceBottle.urdf (robot description, URDF)
Before this commit: robot limeJuice, 2 links, 1 joints
Joints:
- joint body_to_cap: origin xyz=0 0 0.258451 rpy=0 0 0 -> xyz=0 0 0.12923 rpy=0 0 0

File: src/abe_sim/3DObjects/Mango/mango.urdf (robot description, URDF)
Before this commit: robot mango, 2 links, 1 joints
Joints:
- joint man_to_go: origin xyz=0 -0.001 0 rpy=0 0 0 -> xyz=0 -0.0005 0 rpy=0 0 0

File: src/abe_sim/3DObjects/RedWineVinegar/redWineVinegar.urdf (robot description, URDF)
Before this commit: robot vegetableOil, 3 links, 2 joints
Joints:
- joint body_to_cap: origin xyz=0 0 0.546 rpy=0 0 0 -> xyz=0 0 0.273 rpy=0 0 0
- joint body_to_label: origin xyz=0.069 0 0.225 rpy=0 0 0 -> xyz=0.0345 0 0.1225 rpy=0 0 0

File: src/abe_sim/3DObjects/RollingPin/rollingPin.urdf (robot description, URDF)
Before this commit: robot rollingPin, 3 links, 2 joints
Joints:
- joint body_to_grip1: origin xyz=-0.309577 0 0 rpy=0 0 0 -> xyz=-0.154788 0 0 rpy=0 0 0
- joint body_to_grip2: origin xyz=0.309577 0 0 rpy=0 0 0 -> xyz=0.154788 0 0 rpy=0 0 0

File: src/abe_sim/3DObjects/Spatula/spatula.urdf (robot description, URDF)
Before this commit: robot spatula, 2 links, 1 joints
Joints:
- joint grip_to_spatula: origin xyz=-0.231617 0.008735 0 rpy=0 0 0 -> xyz=-0.1158 0.00437 0 rpy=0 0 0

File: src/abe_sim/3DObjects/VegetableOil/vegetableOil.urdf (robot description, URDF)
Before this commit: robot vegetableOil, 3 links, 2 joints
Joints:
- joint body_to_cap: origin xyz=0 0 0.546 rpy=0 0 0 -> xyz=0 0 0.273 rpy=0 0 0
- joint body_to_label: origin xyz=0.069 0 0.225 rpy=0 0 0 -> xyz=0.0345 0 0.1225 rpy=0 0 0

File: src/abe_sim/3DObjects/WhiteVinegar/whiteVinegar.urdf (robot description, URDF)
Before this commit: robot whiteVinegar, 3 links, 2 joints
Joints:
- joint body_to_cap: origin xyz=0 0 0.546 rpy=0 0 0 -> xyz=0 0 0.273 rpy=0 0 0
- joint body_to_label: origin xyz=0.069 0 0.225 rpy=0 0 0 -> xyz=0.0345 0 0.1225 rpy=0 0 0

Commit message: Added remaining base objects
Added bell pepper cube, bell pepper stem, bell pepper strip, bell pepper Seeds, seeded bell pepper, crouton, bread cube, sprinkled bread cube, garlic sprinkled bread cube, red chili pepper strip, cilantro salad dressing bottle + particle, peeled + diced mango, mini marshmallow + bag, milk bag + particle, onion slice, chopped potato, sifted powdered white sugar particle, radish slice, raisin + bag, soaked raisin, chopped Lettuce, lettuce leaf, washed lettuce, chopped rosemary, rosemary sprigs, salt shaker, baked chopped sweet potato, chopped sweet potato, drizzled chopped sweet potato, chopped tomato, half tomato, seeded half tomato, tomato seeds, tomato stem, chopped half walnut, ground walnut

File: src/abe_sim/3DObjects/BellPepper/bellPepper.urdf (robot description, URDF)
Before this commit: robot bellPepper, 2 links, 1 joints
Links:
- link body: geometry collision mesh filename=pepperBodyCollider.obj; visual mesh filename=pepperBody.obj

File: src/abe_sim/3DObjects/Radish/radish.urdf (robot description, URDF)
Before this commit: robot carrot, 2 links, 1 joints
Joints:
- removed joint fruit_to_tail
- added joint body_to_green: type fixed, parent body, child green, origin xyz=0 0 0 rpy=0 0 0

File: src/abe_sim/3DObjects/RomaineLettuce/romaineLettuce.urdf (robot description, URDF)
Before this commit: robot romaineLettuce, 2 links, 1 joints
Links:
- link leaf: geometry collision mesh filename=lettuceCollider.obj; visual mesh filename=lettuceOutside.obj
