Commit message: New version of prefmodel_wrapper_win.py and minor fixed to teaparty assets

File: src/abe_sim/3DObjects/Teaparty/coffeeCup.urdf (robot description, URDF)
Before this commit: robot coffee_cup, 2 links, 1 joints
Joints:
- joint cup_to_coffee: origin xyz=0 0.110023 0 rpy=0 0 0 -> xyz=0 0.12 0 rpy=0 0 0

File: src/abe_sim/3DObjects/Teaparty/coffeeCupMilk.urdf (robot description, URDF)
Before this commit: robot coffee_cup_milk, 2 links, 1 joints
Joints:
- joint cup_to_coffee: origin xyz=0 0.110023 0 rpy=0 0 0 -> xyz=0 0.12 0 rpy=0 0 0
